File: Unified_v1.3/Driver.kicad_sch (KiCad schematic)
At the start: 152 parts, among them Q1 FS8205A, Q2 SI2301-TP, Q4 2N7002, U10 PCF8574T, U11 DRV8876PWPR, U12 TB6612FNG, U13 B0505S-1WR3, U14 MT3608, U15 DW01A, U16 TP4056-42-ESOP8, U4 MP1584EN, U5 TPS54531DDA, U6 ISO1050DUB, U7 INA219AxD, U8 MP1584EN, U9 PCF8574T

Commit message: fix: correct feedback dividers, net label, and TEMP pin circuit
- C-01: R36 71.5K → 14K (U8 MP1584EN Vout: 1.92V → 6.51V target 6.5V)
- C-05: R26 37.4K → 52.3K (U5 TPS54531 Vout: 3.79V → 4.98V target 5V)
- H-01: Rename root label PB6_FAN1_PWM → PA6_FAN1_PWM (was wrong pin ref)
- H-06: Add R92 (100K) between TP4056 TEMP pin and GND (was shorted to
  PROG/GND junction, bypassing thermal protection entirely)

Co-Authored-By: Claude Opus 4.6 (1M context) <noreply@anthropic.com>
Parts:
- added R92: 100K, Resistor_SMD:R_0402_1005Metric, symbol Device:R_Small
- R26: value 37.4K -> 52.3K
- R36: value 71.5K -> 14K
Connections:
- net GND: now also R92.2; no longer U16.1 (TEMP)
- new net: R92.1, U16.1 (TEMP)
Changed lines of the file:
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@@
 	(wire
 		(pts
-			(xy 78.74 281.94) (xy 78.74 284.48)
+			(xy 78.74 281.94) (xy 83.82 281.94)
+		)
+		(stroke
+			(width 0)
+			(type default)
+		)
+	)
+	(wire
+		(pts
+			(xy 88.9 281.94) (xy 88.9 284.48)
 		)
 		(stroke
@@
 			)
 		)
-		(property "Value" "71.5K"
+		(property "Value" "14K"
 			(at 130.556 93.98 0)
 			(effects
@@
 			)
 		)
-		(property "Value" "37.4K"
+		(property "Value" "52.3K"
 			(at 390.144 46.99 0)
 			(effects
@@
 					(unit 1)
 				)
+			)
+		)
+	)
+	(symbol
+		(lib_id "Device:R_Small")
+		(at 86.36 281.94 90)
+		(unit 1)
+		(exclude_from_sim no)
+		(in_bom yes)
+		(on_board yes)
+		(dnp no)
+		(property "Reference" "R92"
+			(at 84.582 280.162 90)
+			(effects
+				(font
+					(size 0.8 0.8)
+				)
+				(justify left)
+			)
+		)
+		(property "Value" "100K"
+			(at 85.09 281.94 90)
+			(effects
+				(font
+					(size 0.8 0.8)
+				)
+				(justify left)
+			)
+		)
+		(property "Footprint" "Resistor_SMD:R_0402_1005Metric"
+			(at 86.36 281.94 0)
+			(effects
+				(font
+					(size 1.27 1.27)
+				)
+				(hide yes)
+			)
+		)
+		(property "Datasheet" "~"
+			(at 86.36 281.94 0)
+			(effects
+				(font
+					(size 1.27 1.27)
+				)
+				(hide yes)
+			)
+		)
+		(property "Description" "Resistor, small symbol"
+			(at 86.36 281.94 0)
+			(effects
+				(font
+					(size 1.27 1.27)
+				)
+				(hide yes)
+			)
+		)
+		(pin "1"
+		)
+		(pin "2"
+		)
+		(instances
+			(project "Unified_v1"
+				(path "/6562dc13-90d6-4c41-9f04-257b733d6416/db3a805b-509d-4f0f-8aaa-0219eafd0d17"
+					(reference "R92")
+					(unit 1)
+				)
+			)
+		)
+	)
+	(symbol
+		(lib_id "power:GND")
+		(at 88.9 284.48 0)
+		(unit 1)
+		(exclude_from_sim no)
+		(in_bom yes)
+		(on_board yes)
+		(dnp no)
+		(fields_autoplaced yes)
+		(property "Reference" "#PWR0201"
+			(at 88.9 290.83 0)
+			(effects
+				(font
+					(size 1.27 1.27)
+				)
+				(hide yes)
+			)
+		)
+		(property "Value" "GND"
+			(at 88.9 289.56 0)
+			(effects
+				(font
+					(size 1.27 1.27)
+				)
+			)
+		)
+		(property "Footprint" ""
+			(at 88.9 284.48 0)
+			(effects
+				(font
+					(size 1.27 1.27)
+				)
+				(hide yes)
+			)
+		)
+		(property "Datasheet" ""
+			(at 88.9 284.48 0)
+			(effects
+				(font
+					(size 1.27 1.27)
+				)
+				(hide yes)
+			)
+		)
+		(property "Description" "Power symbol creates a global label with name \"GND\" , ground"
+			(at 88.9 284.48 0)
+			(effects
+				(font
+					(size 1.27 1.27)
+				)
+				(hide yes)
+			)
+		)
+		(pin "1"
+		)
+		(instances
+			(project "Unified_v1"
+				(path "/6562dc13-90d6-4c41-9f04-257b733d6416/db3a805b-509d-4f0f-8aaa-0219eafd0d17"
+					(reference "#PWR0201")
+					(unit 1)
+				)
